File: guilty-pad-gay.kicad_sch (KiCad schematic)
At the start: 17 parts, among them J1 Conn_01x04_Pin, J2 Conn_01x03_Socket, J3 Conn_01x03_Socket, SW1 SW_Push, SW2 SW_Push, SW3 SW_Push, SW4 SW_Push, U1 XIAO-RP2040-DIP

Commit message: switch to nrf, add boost converter stuff for running LEDs off battery, and update the README
Parts:
- removed D6: 1N4001, Diode_THT:D_DO-41_SOD81_P10.16mm_Horizontal, symbol Diode:1N4001
- removed J1: Conn_01x04_Pin, magnetopad:PinSocket_1x04_P1.8mm_Vertical, symbol Connector:Conn_01x04_Pin
- removed U1: XIAO-RP2040-DIP, OPL:XIAO-RP2040-DIP, symbol OPL:XIAO-RP2040-DIP
- added C2: 1μF, Capacitor_SMD:C_0201_0603Metric_Pad0.64x0.40mm_HandSolder, symbol Device:C
- added D1, D2: D, Diode_SMD:D_SOD-123, symbol Device:D
- added L1: 15μH, Inductor_SMD_Wurth:L_Wurth_WE-LQSH-4020, symbol Device:L
- added Q1: DMC3071LVT, Package_TO_SOT_SMD:TSOT-23-6_HandSoldering, symbol Transistor_FET:DMC3071LVT
- added R1: 806k, Resistor_SMD:R_0402_1005Metric_Pad0.72x0.64mm_HandSolder, symbol Device:R
- added R2: 2M, Resistor_SMD:R_0402_1005Metric_Pad0.72x0.64mm_HandSolder, symbol Device:R
- added TP1, TP2: TestPoint, TestPoint:TestPoint_Pad_2.0x2.0mm, symbol Connector:TestPoint
- added U1: XIAO-nRF52840-SMD, OPL:XIAO-nRF52840-SMD, symbol OPL:XIAO-nRF52840-SMD
- added U2: H8118A40PR, Package_TO_SOT_SMD:SOT-89-3_Handsoldering, symbol guilty-pad-gay:QX2303L40E
Connections:
- net +5V: now also D2.2 (A), Q1.3 (G), U1.14 (5V); no longer J2.1 (Pin_1), LED1.1 (VDD), LED2.1 (VDD), LED3.1 (VDD), LED4.1 (VDD)
- net GND: now also Q1.5 (S), R2.2, TP2.1, U1.13 (GND), U1.16 (GND); no longer J2.3 (Pin_3), LED1.4 (VSS), LED2.4 (VSS), LED3.4 (VSS), LED4.4 (VSS)
- net at SW2.2: now also U1.2 (P0.03_A1_D1)
- net at SW3.2: now also U1.3 (P0.28_A2_D2)
- net at LED1.3 (DIN): now also U1.8 (P1.12_D7_RX)
- net at SW1.2: now also U1.1 (P0.02_A0_D0)
- net at SW4.2: now also U1.4 (P0.29_A3_D3)
- net +5V_LED_board renamed +4_OR_5V_LED_board
- new net: D1.2 (A), U2.2 (VO)
- new net: Q1.4 (D), U2.1 (GND)
- new net: L1.2, U2.3 (VI)
- new net +4_OR_5V: C2.2, D1.1 (K), D2.1 (K), J2.1 (Pin_1), LED1.1 (VDD), LED2.1 (VDD), LED3.1 (VDD), LED4.1 (VDD)
- new net BT_PIN: R1.2, R2.1, U1.5 (P0.04_A4_D4_SDA)
- new net LED_ENABLE: Q1.1 (G), U1.9 (P1.13_D8_SCK)
- new net LED_GND: C2.1, J2.3 (Pin_3), LED1.4 (VSS), LED2.4 (VSS), LED3.4 (VSS), LED4.4 (VSS), Q1.2 (S), Q1.6 (D)
- new net VBAT: L1.1, R1.1, TP1.1, U1.15 (BAT)
Other:
- note added: "NOTE regarding 4/5V rail This is exclusively used for powering the LEDs, which can run off a range of voltages For this we're using 4/5V, but anything 3.7-5.5 works (although DIN must be >= 0.7*VDD, so max VDD in this case is actually ~4.7V) Anyways yeah, +4_OR_5V means 4V when on battery, 5V when on USB"
- note added: "The XIAO nrf52840 only supplies 5V when on USB When on battery, we'll use a boost converter set to 4V (fulfills 3.3V >= 0.7*VDD_LED and 3.8V >= .95*VDD_LED) (those are to cover min LED data voltage relative to VDD, and ensure the boost converter's input voltage is always less than the output) alt boost converter: https://www.lcsc.com/datasheet/C2974847.pdf may be a little more efficient and highe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"
- note added: "boost conversion and LED control circuitry"
- note added: "connector for batt & voltage divider"
- note added: "left LED bank is for backlighting right LED bank is second set of LEDs off to the right not connected to normal power symbols so they don't auto-connect to the rest of the board"
- note removed: "left LED bank is for backlighting right LED bank is second set of LEDs off to the right as always VDD is 5V, GND is VSS not connected to power symbols so they don't auto-connect to the rest of the board"
- note removed: "pogo pins go here pins 2 and 3 (GPIO 0/1) for UART for comm with keyboard pins 1 and 4 for GND and 5V"
