File: guilty-pad-gay.kicad_sch (KiCad schematic)
At the start: 25 parts, among them J2 Conn_01x03_Socket, J3 Conn_01x03_Socket, Q1 DMC3071LVT, SW1 SW_Push, SW2 SW_Push, SW3 SW_Push, SW4 SW_Push, U1 XIAO-nRF52840-SMD, U2 H8118A40PR

Commit message: swap out the capacitor for a bigger one - can use it for both this and the full-size board
Parts:
- C2: value 1μF -> 10μF; footprint Capacitor_SMD:C_0201_0603Metric_Pad0.64x0.40mm_HandSolder -> Capacitor_SMD:C_0603_1608Metric_Pad1.08x0.95mm_HandSolder
Changed lines of the file:
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@@
 			)
 		)
-		(property "Value" "1μF"
+		(property "Value" "10μF"
 			(at 69.85 161.2899 0)
 			(effects
@@
 			)
 		)
-		(property "Footprint" "Capacitor_SMD:C_0201_0603Metric_Pad0.64x0.40mm_HandSolder"
+		(property "Footprint" "Capacitor_SMD:C_0603_1608Metric_Pad1.08x0.95mm_HandSolder"
 			(at 65.0748 156.21 0)
 			(effects

Commit message: swap to 5V and use level shifter - much more sane
Parts:
- added U3: 74LV1T08GW, Package_TO_SOT_SMD:SOT-353_SC-70-5, symbol 74xx:74LV1T08GW
Connections:
- net +4_OR_5V is gone; now on net +5V: C2.2, D1.1 (K), D2.1 (K), J2.1 (Pin_1), LED1.1 (VDD), LED2.1 (VDD), LED3.1 (VDD), LED4.1 (VDD)
- net +5V: now also U3.5 (VCC); no longer D2.2 (A), Q1.3 (G), U1.14 (5V)
- net BT_PIN: now also U1.6 (P0.05_A5_D5_SCL); no longer U1.5 (P0.04_A4_D4_SDA)
- net GND: now also U3.3 (GND)
- net LED_ENABLE: now also U1.7 (P1.11_D6_TX); no longer U1.9 (P1.13_D8_SCK)
- net at U1.8 (P1.12_D7_RX): now also U3.1 (B), U3.2 (A); no longer LED1.3 (DIN)
- new net +5V_USB: D2.2 (A), Q1.3 (G), U1.14 (5V)
- new net LED_CONTROL: LED1.3 (DIN), U3.4 (Y)

Commit message: i forgor to swap out text, that's all
Other:
- note added: "The XIAO nrf52840 only supplies 5V when on USB"
- note removed: "NOTE regarding 4/5V rail This is exclusively used for powering the LEDs, which can run off a range of voltages For this we're using 4/5V, but anything 3.7-5.5 works (although DIN must be >= 0.7*VDD, so max VDD in this case is actually ~4.7V) Anyways yeah, +4_OR_5V means 4V when on battery, 5V when on USB"
- note removed: "The XIAO nrf52840 only supplies 5V when on USB When on battery, we'll use a boost converter set to 4V (fulfills 3.3V >= 0.7*VDD_LED and 3.8V >= .95*VDD_LED) (those are to cover min LED data voltage relative to VDD, and ensure the boost converter's input voltage is always less than the output) alt boost converter: https://www.lcsc.com/datasheet/C2974847.pdf may be a little more efficient and highe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"
Changed lines of the file:
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@@
 	(paper "A4")
-	(rectangle
-		(start 142.494 22.606)
-		(end 275.59 46.99)
-		(stroke
-			(width 0.508)
-			(type default)
-			(color 255 0 0 1)
-		)
-		(fill
-			(type none)
-		)
-	)
 	(rectangle
 		(start 17.78 146.05)
@@
 		)
 	)
-	(text "NOTE regarding 4/5V rail\nThis is exclusively used for powering the LEDs, which can run off a range of voltages\nFor this we're using 4/5V, but anything 3.7-5.5 works\n(although DIN must be >= 0.7*VDD, so max VDD in this case is actually ~4.7V)\n\nAnyways yeah, +4_OR_5V means 4V when on battery, 5V when on USB"
-		(exclude_from_sim no)
-		(at 209.042 34.544 0)
-		(effects
-			(font
-				(size 1.905 1.905)
-			)
-		)
-	)
 	(text "boost conversion and LED control circuitry"
 		(exclude_from_sim no)
@@
 		)
 	)
-	(text "The XIAO nrf52840 only supplies 5V when on USB\nWhen on battery, we'll use a boost converter set to 4V (fulfills 3.3V >= 0.7*VDD_LED and 3.8V >= .95*VDD_LED)\n(those are to cover min LED data voltage relative to VDD,\nand ensure the boost converter's input voltage is always less than the output)\n\nalt boost converter: https://www.lcsc.com/datasheet/C2974847.pdf\nmay be a little more efficient and higher amperage,\nbut more work and more components - will accept the tradeoff to make this simpler"
+	(text "The XIAO nrf52840 only\nsupplies 5V when on USB"
 		(exclude_from_sim no)
-		(at 51.816 139.446 0)
+		(at 70.104 192.024 0)
 		(effects
 			(font
