File: PCB/guilty-pad-gay.kicad_pcb (KiCad board)
At the start: 2 copper layers, 93.8 x 37.1 mm, 34 parts, among them J2 Conn_01x03_Socket, J3 Conn_01x03_Socket, Q1 DMC3071LVT, SW1 SW_Push, SW2 SW_Push, SW3 SW_Push, SW4 SW_Push, U1 XIAO-nRF52840-SMD, U2 H8118A40PR, U3 74LV1T08GW

Commit message: look idek i just want this in git
Parts:
- removed C2: 10μF, Capacitor_SMD:C_0603_1608Metric_Pad1.08x0.95mm_HandSolder
- removed D1, D2: D, Diode_SMD:D_SOD-123
- removed J2, J3: Conn_01x03_Socket, Connector_PinHeader_2.54mm:PinHeader_1x03_P2.54mm_Vertical
- removed L1: 15μH, Inductor_SMD_Wurth:L_Wurth_WE-LQSH-4020
- removed LED1, LED2, LED3, LED4, LED5, LED6, LED7, LED8: SK6812MINI-E, marbastlib-various:LED_6028R
- removed Q1: DMC3071LVT, Package_TO_SOT_SMD:TSOT-23-6_HandSoldering
- removed R1: 806k, Resistor_SMD:R_0402_1005Metric_Pad0.72x0.64mm_HandSolder
- removed R2: 2M, Resistor_SMD:R_0402_1005Metric_Pad0.72x0.64mm_HandSolder
- removed REF** (x2): MouseBite-Slot_2.0x4.5mm_inset_D0.5mm_P0.85mm_7h, Panelization:MouseBite-Slot_2.0x4.5mm_inset_D0.5mm_P0.85mm_7h
- removed SW1, SW2, SW3, SW4: SW_Push, Button_Switch_Keyboard:SW_Cherry_MX_1.00u_PCB
- removed TP1, TP2: TestPoint, TestPoint:TestPoint_Pad_2.0x2.0mm
- removed U1: XIAO-nRF52840-SMD, OPL:XIAO-nRF52840-SMD
- removed U2: H8118A40PR, Package_TO_SOT_SMD:SOT-89-3_Handsoldering
- removed U3: 74LV1T08GW, Package_TO_SOT_SMD:SOT-353_SC-70-5
- moved G*** 55.7 mm to (42.0, 127.2)
- moved G*** 52.1 mm to (76.0, 116.9)
- moved G*** 52.1 mm to (97.7, 102.6)
- moved G*** 52.1 mm to (143.9, 109.1)
- moved G*** 52.1 mm to (69.9, 117.2)
- moved G*** 52.1 mm to (117.8, 116.9)
Routing:
- net /LED_GND: track 182.0 -> 0.00 mm, vias 1 -> 0
- net +5V: track 147.5 -> 0.00 mm, vias 2 -> 0
- net GND: track 132.7 -> 0.00 mm
- net /VBAT: track 100.5 -> 0.00 mm, vias 4 -> 0
- net /LED_CONTROL: track 89.1 -> 0.00 mm, vias 1 -> 0
- net /BT_PIN: track 73.5 -> 0.00 mm, vias 2 -> 0
- net +5V_USB: track 67.7 -> 0.00 mm, vias 2 -> 0
- net Net-(U1-P0.02_A0_D0): track 67.1 -> 0.00 mm
- net Net-(U1-P0.03_A1_D1): track 49.9 -> 0.00 mm
- net /LED_ENABLE: track 39.5 -> 0.00 mm, vias 2 -> 0
- net Net-(J2-Pin_2): track 30.4 -> 0.00 mm, vias 1 -> 0
- net Net-(U1-P0.28_A2_D2): track 27.9 -> 0.00 mm
- net GND_LED_board: track 27.3 -> 0.00 mm, vias 1 -> 0
- net +4_OR_5V_LED_board: track 24.5 -> 0.00 mm, vias 2 -> 0
- net Net-(U2-VI): track 21.6 -> 0.00 mm
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Other:
- board outline removed
