File: PCB/guilty-pad-gay.kicad_pcb (KiCad board)
At the start: 2 copper layers, 135 x 19.9 mm, 40 parts, among them J1 Conn_01x03, J2 Conn_01x04, Q1 AO3400A, Q2 AO3401A, SW1 SW_Push, SW2 SW_Push, SW3 SW_Push, SW4 SW_Push, SW5 SW_Push, SW6 SW_Push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

Commit message: add BOM and update image
Parts:
- D3, D4, D5, D6, D7, D8, G***: moved to F.Cu
- G***, LED1, LED2, LED3, LED4, LED5, LED6: moved to B.Cu
- moved G*** 203.3 mm to (238.8, 76.3), turned to 90 degrees
- moved G*** 89.2 mm to (202.2, 73.3), turned to 0 degrees
- moved G*** 51.8 mm to (113.6, 68.7), turned to 90 degrees
- moved G*** 7.83 mm to (179.9, 73.0)
- moved G*** 0.57 mm to (222.6, 69.4), turned to 180 degrees
- moved D3 0.50 mm to (144.5, 68.0)
- moved D4 0.50 mm to (201.7, 68.0)
- moved D5 0.50 mm to (163.6, 68.0)
- moved D6 0.50 mm to (220.7, 68.0)
- moved D7 0.50 mm to (182.6, 68.0)
- moved D8 0.50 mm to (239.8, 68.0)
- turned U1 to -90 degrees
Routing:
- net /COL0: track 286.3 -> 55.8 mm, vias 5 -> 1
- net /COL1: track 319.4 -> 115.9 mm, vias 2 -> 1
- net Net-(D4-A): track 69.1 -> 11.6 mm
- net Net-(D6-A): track 69.1 -> 12.8 mm
- net Net-(D8-A): track 69.1 -> 13.0 mm
- net Net-(D7-A): track 69.1 -> 13.0 mm
- net Net-(D3-A): track 69.1 -> 13.0 mm
- net Net-(D5-A): track 69.1 -> 13.0 mm
- net /LED_CONTROL: track 13.0 -> 45.7 mm
- net Net-(U1-P1.12_D7_RX): track 26.7 -> 2.60 mm
- net /BATT_LVL: track 6.32 -> 27.6 mm, vias 1 -> 5
- net /ROW2: track 134.4 -> 153.7 mm, vias 2 -> 5
- net /SWDIO: track 21.7 -> 4.11 mm, vias 3 -> 1
- net /ROW1: track 134.4 -> 118.8 mm, vias 2 -> 5
- net /I2C_SCL: track 19.7 -> 4.41 mm
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Other:
- board size 135 x 19.9 mm -> 133.8 x 19.4 mm
