File: PCB/guilty-pad-gay.kicad_sch (KiCad schematic)
At the start: 32 parts, among them Q1 AO3400A, SW1 SW_Push, SW2 SW_Push, SW3 SW_Push, SW5 SW_Push, SW6 SW_Push, SW7 SW_Push, U1 XIAO-nRF52840-SMD, U2 TPS613222ADBV, U3 74LV1T08GW

Commit message: look idr what's different but uh yeag i'm committing
Parts:
- removed D10, D9: D_Small, symbol KiCad:D_Small
- added J1: Conn_01x03, symbol KiCad:Conn_01x03
- added J2: Conn_01x04, symbol KiCad:Conn_01x04
- added Q2: AO3401A, Package_TO_SOT_SMD:SOT-23, symbol KiCad:AO3401A
- added R3: 1M, symbol KiCad:R_Small
Connections:
- net +BATT: now also Q2.3 (D); no longer L1.1
- net GND: now also J1.1 (Pin_1), J2.1 (Pin_1), R3.1
- net LED_CONTROL: now also U1.2 (P0.03_A1_D1)
- net LED_ENABLE: now also Q1.1 (G)
- net VBUS: now also Q2.1 (G), R3.2
- net +3V3: now reaches U1.12 (3V3)
- net +3V3: now also J2.2 (Pin_2)
- net SWDIO: now reaches U1.19 (PA31_SWDIO)
- net SWDIO: now also J1.3 (Pin_3)
- net SWCLK: now reaches U1.20 (PA30_SWCLK)
- net SWCLK: now also J1.2 (Pin_2)
- net I2C_SDA: now reaches U1.5 (P0.04_A4_D4_SDA)
- net I2C_SDA: now also J2.4 (Pin_4)
- net I2C_SCL: now reaches U1.6 (P0.05_A5_D5_SCL)
- net I2C_SCL: now also J2.3 (Pin_3)
- new net: L1.1, Q2.2 (S)
Other:
- note added: "AO3401A Vgs threshold is too low must use NMOS too, rather than another PMOS"
- note added: "TODO: add connectors for i2c and power, and whatever spare pins if possible and also for SWD/GND"
- note removed: "TODO: add connectors for i2c and power, and whatever spare pins if possible and also for SWD/RST/GND"
- moved on the sheet: C2, D1, L1, Q1, U2, U3

Commit message: update with routed and parts and stuffs
Parts:
- removed SW7: SW_Push, Button_Switch_Keyboard:SW_Cherry_MX_1.00u_PCB, symbol Switch:SW_Push
- added SW4: SW_Push, Button_Switch_Keyboard:SW_Cherry_MX_1.00u_PCB, symbol Switch:SW_Push
- D1, D2: footprint Diode_SMD:D_SMA_Handsoldering -> Diode_SMD:D_SOD-323_HandSoldering
- D3, D4, D5, D6, D7, D8: footprint (none) -> Diode_SMD:D_SOD-323_HandSoldering
- J1: footprint (none) -> Connector_JST:JST_GH_SM03B-GHS-TB_1x03-1MP_P1.25mm_Horizontal
- J2: footprint (none) -> Connector_JST:JST_GH_SM04B-GHS-TB_1x04-1MP_P1.25mm_Horizontal
- R1, R2: footprint Resistor_SMD:R_0402_1005Metric_Pad0.72x0.64mm_HandSolder -> Resistor_SMD:R_0805_2012Metric_Pad1.20x1.40mm_HandSolder
- R3: value 1M -> 806k; footprint (none) -> Resistor_SMD:R_0805_2012Metric_Pad1.20x1.40mm_HandSolder
Connections:
- net COL1: now also SW4.1
- net at D6.2 (A): now also SW5.2; no longer SW6.2
- net at D4.2 (A): now also SW4.2; no longer SW5.2
- net at D8.2 (A): now also SW6.2
Other:
- note removed: "TODO: add connectors for i2c and power, and whatever spare pins if possible and also for SWD/GND"

Commit message: add BOM and update image
Parts:
- R1, R3: value 806k -> 820k
Changed lines of the file:
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@@
 			)
 		)
-		(property "Value" "806k"
+		(property "Value" "820k"
 			(at 23.114 159.766 0)
 			(show_name no)
@@
 			)
 		)
-		(property "Value" "806k"
+		(property "Value" "820k"
 			(at 36.83 104.902 90)
 			(show_name no)
